Commit message: Squint v1.1.0 - Added image transport node and camera_info topic remapping

File: ardi/urdf/inertial_macros.xacro (robot description, xacro)
@@ -1,8 +1,10 @@
 <?xml version="1.0"?>
+<!-- v1.1.0 - Added image transport node and camera_info topic remapping -->
 <robot xmlns:xacro="http://www.ros.org/wiki/xacro" >
-    <!-- Standard inertial calculations https://en.wikipedia.org/wiki/List_of_moments_of_inertia
-    Based on geometry -->
+    <!-- Some standard inertial calculations https://en.wikipedia.org/wiki/List_of_moments_of_inertia -->
+    <!-- Based on geometry of shape -->
     <xacro:macro name="inertial_sphere" params="mass radius">
         <inertial>
+            <!-- <xacro:insert_block name="origin"/> -->
             <mass value="${mass}" />
             <inertia ixx="${(2/5) * mass * (radius*radius)}" ixy="0.0" ixz="0.0"
@@ -13,4 +15,5 @@
     <xacro:macro name="box_inertia" params="mass x y z">
         <inertial>
+            <!-- <xacro:insert_block name="origin"/> -->
             <mass value="${mass}" />
             <inertia ixx="${(1/12) * mass * (y*y+z*z)}" ixy="0.0" ixz="0.0"
@@ -21,4 +24,5 @@
     <xacro:macro name="cylinder_inertia" params="mass length radius">
         <inertial>
+            <!-- <xacro:insert_block name="origin"/> -->
             <mass value="${mass}" />
             <inertia ixx="${(1/12) * mass * (3*radius*radius + length*length)}" ixy="0.0" ixz="0.0"

File: ardi/urdf/robot_model.urdf (robot description, URDF)
Before this commit: robot ardi, 22 links, 21 joints
Links:
- link imu_link: geometry collision box size=0.03 0.06 0.02; visual box size=0.03 0.06 0.02
